File: Fuente 12V/Fuente 12V.kicad_pcb (KiCad board)
At the start: 2 copper layers, 100 x 50 mm, 17 parts, among them U1 LM7812_TO220, U2 LM7912_TO220

Commit message: Actualizacion de respo Kicad
Parts:
- added REF**: MountingHole_2.2mm_M2, MountingHole:MountingHole_2.2mm_M2, F.Cu at (203.8, 114.8)
- added REF**: MountingHole_2.2mm_M2, MountingHole:MountingHole_2.2mm_M2, F.Cu at (115.5, 75.2)
- added REF**: MountingHole_2.2mm_M2, MountingHole:MountingHole_2.2mm_M2, F.Cu at (115.5, 114.8)
- added REF**: MountingHole_2.2mm_M2, MountingHole:MountingHole_2.2mm_M2, F.Cu at (203.8, 75.5)
Routing:
- net (no net): vias 4 -> 0
- added copper zone on B.Cu, net (none)
- removed copper zone on B.Cu, net Earth
Other:
- net class Default removed
