File: Librerias_KiCad/Raspberry Pico 2 THT/Test/Test.kicad_sch (KiCad schematic)
At the start: 5 parts, among them J1 Conn_01x20, J2 Conn_01x20, J3 Conn_01x03, U1 Pico, U2 RP2350

Commit message: Mejora de Placa de desarrollo
Parts:
- removed U2: RP2350, BoardF_Pi_Pico:BoardF_Pi_Pico_RP2350, symbol Raspberry Pi Pico:Board_Pi_Pico_2350
Connections:
- net GND: no longer J1.13 (Pin_13), J1.18 (Pin_18), J1.8 (Pin_8), J2.13 (Pin_13), J2.18 (Pin_18), J2.3 (Pin_3), J3.2 (Pin_2)
