File: Placa_de_Desarrollo/Placa_de_Desarrollo.kicad_sch (KiCad schematic)
At the start: 27 parts, among them J1 USB_B_Micro, J2 Conn_01x20, J3 ADC0, J4 ADC1, J5 ADC2, J6 Conn_01x14, SW1 RESET, U1 LM317_TO-220, U2 Pico

Commit message: Mejora de Placa de desarrollo
Parts:
- removed J1: USB_B_Micro, Connector_PinHeader_2.54mm:PinHeader_1x06_P2.54mm_Vertical, symbol Connector:USB_B_Micro
- removed J3: ADC0, Connector_PinHeader_2.54mm:PinHeader_1x05_P2.54mm_Vertical, symbol Connector_Generic:Conn_01x05
- removed J4: ADC1, Connector_PinHeader_2.54mm:PinHeader_1x05_P2.54mm_Vertical, symbol Connector_Generic:Conn_01x05
- removed J5: ADC2, Connector_PinHeader_2.54mm:PinHeader_1x05_P2.54mm_Vertical, symbol Connector_Generic:Conn_01x05
- removed U2: Pico, MCU_RaspberryPi_and_Boards:RPi_Pico_SMD_TH, symbol MCU_RaspberryPi_and_Boards:Pico
- added RV2, RV3, RV4: 10k, Potentiometer_THT:Potentiometer_Piher_T-16H_Single_Horizontal, symbol Device:R_Potentiometer
- added U2: RP2350, BoardF_Pi_Pico:BoardF_Pi_Pico_RP2350, symbol Raspberry Pi Pico:Board_Pi_Pico_2350
- added U3: ~, Micro_USB_PCB:Micro_USB_B, symbol Micro_USB_B_PCB:Micro_USB_B
- SW1: footprint Button_Switch_THT:SW_PUSH_6mm_H9.5mm -> Button_Switch_THT:SW_PUSH_6mm
- renumbered J6 to J3
Connections:
- net 3.3V: now also RV2.1, RV3.1, RV4.1
- net 5V: now also U2.39 (VSYS), U3.5 (VBUS)
- net ADC0: now also RV4.2, U2.31 (GPIO26)
- net ADC1: now also RV3.2, U2.32 (GPIO27)
- net ADC2: now also RV2.2, U2.34 (GPIO28)
- net BUZZER: now also U2.29 (GPIO22)
- net C1/GPIO18: now also U2.24 (GPIO18)
- net C2/GPIO19: now also U2.25 (GPIO19)
- net C3/GPIO20: now also U2.26 (GPIO20)
- net C4/GPIO21: now also U2.27 (GPIO21)
- net F1/GPIO14: now also U2.19 (GPIO14)
- net F2/GPIO15: now also U2.20 (GPIO15)
- net F3/GPIO16: now also U2.21 (GPIO16)
- net F4/GPIO17: now also U2.22 (GPIO17)
- net GND: now also J2.13 (Pin_13), J2.18 (Pin_18), J2.3 (Pin_3), J2.8 (Pin_8), J3.12 (Pin_12), J3.2 (Pin_2), RV2.3, RV3.3, RV4.3, U2.13 (GND), U2.18 (GND), U2.23 (GND), U2.28 (GND), U2.3 (GND), U2.33 (GND), U2.38 (GND), U2.42 (GND), U2.8 (GND), U3.1 (GND)
- net GPIO0/SCK: now also U2.1 (GPIO0)
- net GPIO13: now also U2.17 (GPIO13)
- net GPIO1/TX: now also U2.2 (GPIO1)
- net GPIO2/RX: now also U2.4 (GPIO2)
- net GPIO3/CSn: now also U2.5 (GPIO3)
- net GPIO4: now also U2.6 (GPIO4)
- net GPIO5: now also U2.7 (GPIO5)
- net LED1: now also U2.14 (GPIO10)
- net LED2: now also U2.15 (GPIO11)
- net LED3: now also U2.16 (GPIO12)
- net SCL0: now also U2.12 (GPIO9)
- net SCL1: now also U2.10 (GPIO7)
- net SDA0: now also U2.11 (GPIO8)
- net SDA1: now also U2.9 (GPIO6)
- net at SW1.1: now also U2.30 (RUN)
- no-connect marks 24 -> 10
Other:
- note removed: "NOTA3"

Commit message: Version 1.0 finalizada
Parts:
- removed U3: ~, Micro_USB_PCB:Micro_USB_B, symbol Micro_USB_B_PCB:Micro_USB_B
- added J1: USB_A, Connector_USB:USB_A_Molex_67643_Horizontal, symbol Connector:USB_A
- added JP1, JP2, JP3: Jumper_2_Bridged, Connector_PinHeader_2.54mm:PinHeader_1x02_P2.54mm_Vertical, symbol Jumper:Jumper_2_Bridged
- J2: value Conn_01x20 -> LEFT
- J3: value Conn_01x14 -> RIGHT
Connections:
- net 5V: now also J1.1 (VBUS)
- net GND: now also J1.4 (GND), J1.5 (Shield)
- net LED1: now also JP3.1 (A); no longer R10.1
- net LED2: now also JP2.1 (A); no longer R9.1
- net LED3: now also JP1.1 (A); no longer R8.1
- net C1/GPIO18 renamed GPIO18
- net C2/GPIO19 renamed GPIO19
- net C3/GPIO20 renamed GPIO20
- net C4/GPIO21 renamed GPIO21
- net F1/GPIO14 renamed GPIO14
- net F2/GPIO15 renamed GPIO15
- net F3/GPIO16 renamed GPIO16
- net F4/GPIO17 renamed GPIO17
- net GPIO0/SCK renamed GPIO0
- net GPIO1/TX renamed GPIO1
- net GPIO2/RX renamed GPIO2
- net GPIO3/CSn renamed GPIO3
- new net: JP1.2 (B), R8.1
- new net: JP2.2 (B), R9.1
- new net: JP3.2 (B), R10.1
- no-connect marks 10 -> 9
Other:
- note removed: "CONVERSOR ANALOGICO - DIGITAL"
- moved on the sheet: BZ1, J2, J3, R7, RV2, RV3, RV4
