File: Placa_de_Desarrollo/Placa_de_Desarrollo.kicad_pcb (KiCad board)
At the start: 2 copper layers, 115 x 95 mm, 44 parts, among them J1 USB_A, J10 Conn_01x04, J11 Conn_01x03, J12 Conn_01x04, J13 Conn_01x04, J14 Conn_01x04, J15 Conn_01x04, J16 Conn_01x04, J17 Conn_01x01, J18 Conn_01x01, J2 LEFT, J3 RIGHT, J4 Conn_01x01, J5 Conn_01x04, J6 Conn_01x04, J7 Conn_01x04, J8 Conn_01x03, J9 Conn_01x04, Q1 BC547, SW1 RESET, SW2 PULL DOWN, SW3 PULL UP, U2 RP2350

Commit message: Resguardo para actualizar KiCAD a version 10
Routing:
- net GND: track 446.5 -> 448.6 mm
- added copper zone on B.Cu, net GND
Changed lines of the file:
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@@
 		(allow_soldermask_bridges_in_footprints no)
 		(pcbplotparams
-			(layerselection 0x0001030_ffffffff)
+			(layerselection 0x00010f0_ffffffff)
 			(plot_on_all_layers_selection 0x0000000_00000000)
 			(disableapertmacros no)
-			(usegerberextensions no)
-			(usegerberattributes yes)
-			(usegerberadvancedattributes yes)
+			(usegerberextensions yes)
+			(usegerberattributes no)
+			(usegerberadvancedattributes no)
 			(creategerberjobfile yes)
 			(dashed_line_dash_ratio 12.000000)
@@
 			(sketchpadsonfab no)
 			(subtractmaskfromsilk no)
-			(outputformat 4)
+			(outputformat 1)
 			(mirror no)
 			(drillshape 0)
 			(scaleselection 1)
-			(outputdirectory "../../../../")
+			(outputdirectory "../../../../Gerber/")
 		)
 	)
@@
 		(at 158.61 74.1975)
 		(property "Reference" "U2"
-			(at 0 -0.5 0)
+			(at 1.69 0.0025 0)
 			(unlocked yes)
 			(layer "F.SilkS")
@@
 	)
 	(segment
-		(start 175.215 56.4175)
-		(end 195.4825 56.4175)
+		(start 207.459 55.884)
+		(end 198.597 55.884)
 		(width 1)
 		(layer "B.Cu")
@@
 	)
 	(segment
-		(start 207.459 55.884)
-		(end 198.597 55.884)
+		(start 196 55.9)
+		(end 198.533 55.9)
+		(width 1)
+		(layer "B.Cu")
+		(net 2)
+	)
+	(segment
+		(start 198.533 55.9)
+		(end 198.573 55.86)
 		(width 1)
 		(layer "B.Cu")
@@
 	)
 	(segment
-		(start 198.533 55.9)
-		(end 198.573 55.86)
-		(width 1)
-		(layer "B.Cu")
-		(net 2)
-	)
-	(segment
 		(start 158.6 104.25)
 		(end 160.14 104.25)
@@
 	)
 	(segment
-		(start 197.43 43.65)
-		(end 181.71 43.65)
+		(start 175.215 56.4175)
+		(end 179.6175 56.4175)
 		(width 1)
 		(layer "B.Cu")
@@
 	)
 	(segment
-		(start 196 55.9)
-		(end 198.533 55.9)
+		(start 197.43 43.65)
+		(end 181.71 43.65)
 		(width 1)
 		(layer "B.Cu")
@@
 	)
 	(segment
-		(start 195.4825 56.4175)
+		(start 192.9 59)
 		(end 196 55.9)
 		(width 1)
@@
 	)
 	(segment
+		(start 182.2 59)
+		(end 192.9 59)
+		(width 1)
+		(layer "B.Cu")
+		(net 2)
+	)
+	(segment
 		(start 210 75.5)
 		(end 208.832 74.332)
@@
 	)
 	(segment
+		(start 179.6175 56.4175)
+		(end 182.2 59)
+		(width 1)
+		(layer "B.Cu")
+		(net 2)
+	)
+	(segment
 		(start 210 80.8)
 		(end 210 75.5)
@@
 		(net 51)
 	)
+	(zone
+		(net 2)
+		(net_name "GND")
+		(layer "B.Cu")
+		(hatch edge 0.5)
+		(connect_pads yes
+			(clearance 0.5)
+		)
+		(min_thickness 0.25)
+		(filled_areas_thickness no)
+		(fill yes
+			(thermal_gap 0.5)
+			(thermal_bridge_width 0.5)
+			(island_removal_mode 1)
+			(island_area_min 10)
+		)
+		(polygon
+			(pts
+				(xy 107 26) (xy 220 26) (xy 220 119) (xy 107 119)
+			)
+		)
+	)
 )
